Commit message: lite3 can trot in sim

File: model-control/src/robot_description/lite3_description/Lite3White/urdf/Lite3.urdf (robot description, URDF)
Before this commit: robot MiniLiteV3, 18 links, 17 joints
Links:
- link TORSO: geometry collision box size=0.234 0.184 0.08; visual mesh filename=package://lite3_description/meshes/TORSO.dae

File: model-control/src/robot_description/lite3_description/xacro/body.xacro (robot description, xacro)
@@ -33,5 +33,5 @@
       </inertial>
       <visual>
-        <origin rpy="1.5708 0 1.5708" xyz="-0.231 -0.55 0.09"/>
+        <origin rpy="1.5708 0 1.5708" xyz="-0.231 -0.5625 0.08"/>
         <geometry>
           <mesh filename="package://lite3_description/meshes/FL_HIP.dae" />
@@ -53,5 +53,5 @@
       </inertial>
       <visual>
-        <origin rpy="-2.0 0 1.5708" xyz="0.24 -0.66 0.021"/>
+        <origin rpy="-2.0 0 1.5708" xyz="0.265 -0.66 0.011"/>
         <geometry>
           <mesh filename="package://lite3_description/meshes/L_THIGH.dae" />
@@ -79,4 +79,5 @@
       </inertial>
       <visual>
+      <origin xyz="0 0 -0.03"/>
         <geometry>
           <mesh filename="package://lite3_description/meshes/SHANK.dae" />
@@ -86,5 +87,5 @@
         <origin xyz="0 0 -0.09"/>
         <geometry>
-          <box size="0.02 0.02 0.18"/>
+          <box size="0.02 0.02 0.20"/>
         </geometry>
       </collision>
@@ -109,5 +110,5 @@
     </link>
     <joint name="FL_Ankle" type="fixed">
-      <origin xyz="0 0 -0.20"/>
+      <origin xyz="0 0 -0.21"/>
       <parent link="FL_SHANK" />
       <child link="FL_FOOT" />
@@ -120,5 +121,5 @@
       </inertial>
       <visual>
-        <origin rpy="1.5708 0 1.5708" xyz="-0.231 -0.46 0.085"/>
+        <origin rpy="1.5708 0 1.5708" xyz="-0.231 -0.446 0.0835"/>
         <geometry>
           <mesh filename="package://lite3_description/meshes/FR_HIP.dae" />
@@ -140,5 +141,5 @@
       </inertial>
       <visual>
-        <origin rpy="-2.0 0 1.5708" xyz="0.24 -0.35 0.021"/>
+        <origin rpy="-2.0 0 1.5708" xyz="0.265 -0.35 0.011"/>
         <geometry>
           <mesh filename="package://lite3_description/meshes/R_THIGH.dae" />
@@ -166,4 +167,5 @@
       </inertial>
       <visual>
+      <origin xyz="0 0 -0.03"/>
         <geometry>
           <mesh filename="package://lite3_description/meshes/SHANK.dae" />
@@ -173,5 +175,5 @@
         <origin xyz="0 0 -0.09"/>
         <geometry>
-          <box size="0.02 0.02 0.18"/>
+          <box size="0.02 0.02 0.20"/>
         </geometry>
       </collision>
@@ -196,5 +198,5 @@
     </link>
     <joint name="FR_Ankle" type="fixed">
-      <origin xyz="0 0 -0.20"/>
+      <origin xyz="0 0 -0.21"/>
       <parent link="FR_SHANK" />
       <child link="FR_FOOT" />
@@ -207,5 +209,6 @@
       </inertial>
       <visual>
-        <origin rpy="1.5708 0 1.5708" xyz="0.12 -0.55 0.09"/>
+        <origin rpy="1.5708 0 1.5708" xyz="0.12 -0.5625 0.09"/>
+        <!-- <origin rpy="1.5708 0 1.5708" xyz="-0.231 -0.5625 0.08"/> -->
         <geometry>
           <mesh filename="package://lite3_description/meshes/HL_HIP.dae" />
@@ -227,5 +230,5 @@
       </inertial>
       <visual>
-        <origin rpy="-2.0 0 1.5708" xyz="0.24 -0.66 0.021"/>
+        <origin rpy="-2.0 0 1.5708" xyz="0.27 -0.66 0.011"/>
         <geometry>
           <mesh filename="package://lite3_description/meshes/L_THIGH.dae" />
@@ -253,4 +256,5 @@
       </inertial>
       <visual>
+      <origin xyz="0 0 -0.03"/>
         <geometry>
           <mesh filename="package://lite3_description/meshes/SHANK.dae" />
@@ -260,5 +264,5 @@
         <origin xyz="0 0 -0.09"/>
         <geometry>
-          <box size="0.02 0.02 0.18"/>
+          <box size="0.02 0.02 0.20"/>
         </geometry>
       </collision>
@@ -283,5 +287,5 @@
     </link>
     <joint name="HL_Ankle" type="fixed">
-      <origin xyz="0 0 -0.20"/>
+      <origin xyz="0 0 -0.21"/>
       <parent link="HL_SHANK" />
       <child link="HL_FOOT" />
@@ -294,5 +298,5 @@
       </inertial>
       <visual>
-        <origin rpy="1.5708 0 1.5708" xyz="0.12 -0.46 0.09"/>
+        <origin rpy="1.5708 0 1.5708" xyz="0.13 -0.445 0.09"/>
         <geometry>
           <mesh filename="package://lite3_description/meshes/HR_HIP.dae" />
@@ -314,5 +318,5 @@
       </inertial>
       <visual>
-        <origin rpy="-2.0 0 1.5708" xyz="0.24 -0.35 0.021"/>
+        <origin rpy="-2.0 0 1.5708" xyz="0.27 -0.35 0.013"/>
         <geometry>
           <mesh filename="package://lite3_description/meshes/R_THIGH.dae" />
@@ -340,4 +344,5 @@
       </inertial>
       <visual>
+        <origin xyz="0 0 -0.03"/>
         <geometry>
           <mesh filename="package://lite3_description/meshes/SHANK.dae" />
@@ -347,5 +352,5 @@
         <origin xyz="0 0 -0.09"/>
         <geometry>
-          <box size="0.02 0.02 0.18"/>
+          <box size="0.02 0.02 0.20"/>
         </geometry>
       </collision>
@@ -370,5 +375,5 @@
     </link>
     <joint name="HR_Ankle" type="fixed">
-      <origin xyz="0 0 -0.20"/>
+      <origin xyz="0 0 -0.21"/>
       <parent link="HR_SHANK" />
       <child link="HR_FOOT" />
