Commit message: modify the FR_Knee_joint origin in Lite+foot.urdf

File: rl-robotics/legged_gym/resources/robots/lite3/urdf/Lite3+foot.urdf (robot description, URDF)
Before this commit: robot MiniLiteV3, 22 links, 21 joints
Joints:
- joint FL_Knee_joint: origin xyz=0 0 -0.20 -> xyz=0.0 0 -0.18
- joint FR_Knee_joint: origin xyz=0 0 -0.20 -> xyz=0 0 -0.18
- joint HL_Knee_joint: origin xyz=0 0 -0.20 -> xyz=0 0 -0.18
- joint HR_Knee_joint: origin xyz=0 0 -0.20 -> xyz=0 0 -0.18
