Commit message: [demo] add all
Signed-off-by: trantor <postrantor@gmail.com>

File: robot_description/urdf/model.urdf (robot description, URDF)
Before this commit: robot a1_description, 23 links, 22 joints
Links:
- link FL_calf: geometry collision box size=0.2 0.016 0.016; visual mesh filename=package://robot_description/meshes/calf.dae scale=1 1 1
- link FL_hip: geometry collision cylinder length=0.04 radius=0.046; visual mesh filename=package://robot_description/meshes/hip.dae scale=1 1 1
- link FL_thigh: geometry collision box size=0.2 0.0245 0.034; visual mesh filename=package://robot_description/meshes/thigh.dae scale=1 1 1
- link FR_calf: geometry collision box size=0.2 0.016 0.016; visual mesh filename=package://robot_description/meshes/calf.dae scale=1 1 1
- link FR_hip: geometry collision cylinder length=0.04 radius=0.046; visual mesh filename=package://robot_description/meshes/hip.dae scale=1 1 1
- link FR_thigh: geometry collision box size=0.2 0.0245 0.034; visual mesh filename=package://robot_description/meshes/thigh_mirror.dae scale=1 1 1
- link RL_calf: geometry collision box size=0.2 0.016 0.016; visual mesh filename=package://robot_description/meshes/calf.dae scale=1 1 1
- link RL_hip: geometry collision cylinder length=0.04 radius=0.046; visual mesh filename=package://robot_description/meshes/hip.dae scale=1 1 1
- link RL_thigh: geometry collision box size=0.2 0.0245 0.034; visual mesh filename=package://robot_description/meshes/thigh.dae scale=1 1 1
- link RR_calf: geometry collision box size=0.2 0.016 0.016; visual mesh filename=package://robot_description/meshes/calf.dae scale=1 1 1
- link RR_hip: geometry collision cylinder length=0.04 radius=0.046; visual mesh filename=package://robot_description/meshes/hip.dae scale=1 1 1
- link RR_thigh: geometry collision box size=0.2 0.0245 0.034; visual mesh filename=package://robot_description/meshes/thigh_mirror.dae scale=1 1 1
- link trunk: geometry collision box size=0.267 0.194 0.114; visual mesh filename=package://robot_description/meshes/trunk.dae scale=1 1 1

File: robot_description/xacro/const.xacro (robot description, xacro)
@@ -1,5 +1,6 @@
 <?xml version="1.0"?>
-<robot name="a1_description" xmlns:xacro="http://www.ros.org/wiki/xacro">
-    <!-- Constants for robot dimensions -->
+<robot name="a1_description"
+    xmlns:xacro="http://www.ros.org/wiki/xacro">
+    <!-- constants for robot dimensions -->
     <xacro:property name="PI" value="3.1415926535897931"/>
     <xacro:property name="stick_mass" value="0.00001"/>

File: robot_description/xacro/gazebo.xacro (robot description, xacro)
@@ -40,5 +40,5 @@
         </plugin>
     </gazebo> -->
-   <!-- <gazebo>
+    <!-- <gazebo>
        <plugin filename="libgazebo_ros_force.so" name="gazebo_ros_force">
            <bodyName>trunk</bodyName>
@@ -68,39 +68,39 @@
     <gazebo reference="FR_calf">
         <sensor name="FR_foot_contact" type="contact">
-        <update_rate>100</update_rate>
-        <plugin name="contactPlugin" filename="libunitreeFootContactPlugin.so"/>
-        <contact>
-            <collision>FR_calf_fixed_joint_lump__FR_foot_collision_1</collision>
-        </contact>
+            <update_rate>100</update_rate>
+            <plugin name="contactPlugin" filename="libunitreeFootContactPlugin.so"/>
+            <contact>
+                <collision>FR_calf_fixed_joint_lump__FR_foot_collision_1</collision>
+            </contact>
         </sensor>
     </gazebo>
     <gazebo reference="FL_calf">
         <sensor name="FL_foot_contact" type="contact">
-        <update_rate>100</update_rate>
-        <plugin name="contactPlugin" filename="libunitreeFootContactPlugin.so"/>
-        <contact>
-            <collision>FL_calf_fixed_joint_lump__FL_foot_collision_1</collision>
-        </contact>
+            <update_rate>100</update_rate>
+            <plugin name="contactPlugin" filename="libunitreeFootContactPlugin.so"/>
+            <contact>
+                <collision>FL_calf_fixed_joint_lump__FL_foot_collision_1</collision>
+            </contact>
         </sensor>
     </gazebo>
     <gazebo reference="RR_calf">
         <sensor name="RR_foot_contact" type="contact">
-        <update_rate>100</update_rate>
-        <plugin name="contactPlugin" filename="libunitreeFootContactPlugin.so"/>
-        <contact>
-            <collision>RR_calf_fixed_joint_lump__RR_foot_collision_1</collision>
-        </contact>
+            <update_rate>100</update_rate>
+            <plugin name="contactPlugin" filename="libunitreeFootContactPlugin.so"/>
+            <contact>
+                <collision>RR_calf_fixed_joint_lump__RR_foot_collision_1</collision>
+            </contact>
         </sensor>
     </gazebo>
     <gazebo reference="RL_calf">
         <sensor name="RL_foot_contact" type="contact">
-        <update_rate>100</update_rate>
-        <plugin name="contactPlugin" filename="libunitreeFootContactPlugin.so"/>
-        <contact>
-            <collision>RL_calf_fixed_joint_lump__RL_foot_collision_1</collision>
-        </contact>
-        </sensor>
-    </gazebo>
-    <!-- Visualization of Foot contacts. -->
+            <update_rate>100</update_rate>
+            <plugin name="contactPlugin" filename="libunitreeFootContactPlugin.so"/>
+            <contact>
+                <collision>RL_calf_fixed_joint_lump__RL_foot_collision_1</collision>
+            </contact>
+        </sensor>
+    </gazebo>
+    <!-- visualization of foot contacts. -->
     <!-- <gazebo reference="FR_foot">
         <visual>
@@ -132,5 +132,5 @@
     </gazebo> -->
     <!-- Show planned pose location -->
-     <!-- <gazebo reference="base">
+    <!-- <gazebo reference="base">
         <visual>
             <plugin name="drawLinesPlugin" filename="libdrawLinesPlugin.so">
@@ -146,6 +146,6 @@
         <mu1>0.2</mu1>
         <mu2>0.2</mu2>
-        <kp  value="1000000.0"/>
-        <kd  value="1.0"/>
+        <kp value="1000000.0"/>
+        <kd value="1.0"/>
     </gazebo>
     <gazebo reference="stick_link">
@@ -170,6 +170,6 @@
         <self_collide>1</self_collide>
         <material>Gazebo/DarkGrey</material>
-        <kp  value="1000000.0"/>
-        <kd  value="1.0"/>
+        <kp value="1000000.0"/>
+        <kd value="1.0"/>
     </gazebo>
     <gazebo reference="FL_calf">
@@ -183,6 +183,6 @@
         <self_collide>1</self_collide>
         <material>Gazebo/DarkGrey</material>
-        <kp  value="1000000.0"/>
-        <kd  value="1.0"/>
+        <kp value="1000000.0"/>
+        <kd value="1.0"/>
     </gazebo>
     <!-- FR leg -->
@@ -197,6 +197,6 @@
         <self_collide>1</self_collide>
         <material>Gazebo/DarkGrey</material>
-        <kp  value="1000000.0"/>
-        <kd  value="1.0"/>
+        <kp value="1000000.0"/>
+        <kd value="1.0"/>
     </gazebo>
     <gazebo reference="FR_calf">
@@ -210,6 +210,6 @@
         <self_collide>1</self_collide>
         <material>Gazebo/DarkGrey</material>
-        <kp  value="1000000.0"/>
-        <kd  value="1.0"/>
+        <kp value="1000000.0"/>
+        <kd value="1.0"/>
     </gazebo>
     <!-- RL leg -->
@@ -224,6 +224,6 @@
         <self_collide>1</self_collide>
         <material>Gazebo/DarkGrey</material>
-        <kp  value="1000000.0"/>
-        <kd  value="1.0"/>
+        <kp value="1000000.0"/>
+        <kd value="1.0"/>
     </gazebo>
     <gazebo reference="RL_calf">
@@ -237,6 +237,6 @@
         <self_collide>1</self_collide>
         <material>Gazebo/DarkGrey</material>
-        <kp  value="1000000.0"/>
-        <kd  value="1.0"/>
+        <kp value="1000000.0"/>
+        <kd value="1.0"/>
     </gazebo>
     <!-- RR leg -->
@@ -251,6 +251,6 @@
         <self_collide>1</self_collide>
         <material>Gazebo/DarkGrey</material>
-        <kp  value="1000000.0"/>
-        <kd  value="1.0"/>
+        <kp value="1000000.0"/>
+        <kd value="1.0"/>
     </gazebo>
     <gazebo reference="RR_calf">
@@ -264,6 +264,6 @@
         <self_collide>1</self_collide>
         <material>Gazebo/DarkGrey</material>
-        <kp  value="1000000.0"/>
-        <kd  value="1.0"/>
+        <kp value="1000000.0"/>
+        <kd value="1.0"/>
     </gazebo>
 </robot>

File: robot_description/xacro/leg.xacro (robot description, xacro)
@@ -1,5 +1,5 @@
 <?xml version="1.0"?>
 <robot xmlns:xacro="http://www.ros.org/wiki/xacro">
-    <xacro:include filename="$(find a1_description)/xacro/transmission.xacro"/>
+    <xacro:include filename="$(find robot_description)/xacro/transmission.xacro"/>
     <!-- <xacro:property name="damping" value="0.3" />
     <xacro:property name="friction" value="0.3" /> -->
@@ -33,5 +33,5 @@
                 </xacro:if>
                 <geometry>
-                    <mesh filename="package://a1_description/meshes/hip.dae" scale="1 1 1"/>
+                    <mesh filename="package://robot_description/meshes/hip.dae" scale="1 1 1"/>
                 </geometry>
                 <material name="orange"/>
@@ -46,8 +46,5 @@
                 <origin rpy="0 0 0" xyz="${hip_com_x*front_hind} ${hip_com_y*mirror} ${hip_com_z}"/>
                 <mass value="${hip_mass}"/>
-                <inertia
-                    ixx="${hip_ixx}" ixy="${hip_ixy*mirror*front_hind}" ixz="${hip_ixz*front_hind}"
-                    iyy="${hip_iyy}" iyz="${hip_iyz*mirror}"
-                    izz="${hip_izz}"/>
+                <inertia ixx="${hip_ixx}" ixy="${hip_ixy*mirror*front_hind}" ixz="${hip_ixz*front_hind}" iyy="${hip_iyy}" iyz="${hip_iyz*mirror}" izz="${hip_izz}"/>
             </inertial>
         </link>
@@ -79,8 +76,8 @@
                 <geometry>
                     <xacro:if value="${mirror_dae == True}">
-                        <mesh filename="package://a1_description/meshes/thigh.dae" scale="1 1 1"/>
+                        <mesh filename="package://robot_description/meshes/thigh.dae" scale="1 1 1"/>
                     </xacro:if>
                     <xacro:if value="${mirror_dae == False}">
-                        <mesh filename="package://a1_description/meshes/thigh_mirror.dae" scale="1 1 1"/>
+                        <mesh filename="package://robot_description/meshes/thigh_mirror.dae" scale="1 1 1"/>
                     </xacro:if>
                 </geometry>
@@ -96,8 +93,5 @@
                 <origin rpy="0 0 0" xyz="${thigh_com_x} ${thigh_com_y*mirror} ${thigh_com_z}"/>
                 <mass value="${thigh_mass}"/>
-                <inertia
-                    ixx="${thigh_ixx}" ixy="${thigh_ixy*mirror}" ixz="${thigh_ixz}"
-                    iyy="${thigh_iyy}" iyz="${thigh_iyz*mirror}"
-                    izz="${thigh_izz}"/>
+                <inertia ixx="${thigh_ixx}" ixy="${thigh_ixy*mirror}" ixz="${thigh_ixz}" iyy="${thigh_iyy}" iyz="${thigh_iyz*mirror}" izz="${thigh_izz}"/>
             </inertial>
         </link>
@@ -114,5 +108,5 @@
                 <origin rpy="0 0 0" xyz="0 0 0"/>
                 <geometry>
-                    <mesh filename="package://a1_description/meshes/calf.dae" scale="1 1 1"/>
+                    <mesh filename="package://robot_description/meshes/calf.dae" scale="1 1 1"/>
                 </geometry>
                 <material name="orange"/>
@@ -127,8 +121,5 @@
                 <origin rpy="0 0 0" xyz="${calf_com_x} ${calf_com_y} ${calf_com_z}"/>
                 <mass value="${calf_mass}"/>
-                <inertia
-                    ixx="${calf_ixx}" ixy="${calf_ixy}" ixz="${calf_ixz}"
-                    iyy="${calf_iyy}" iyz="${calf_iyz}"
-                    izz="${calf_izz}"/>
+                <inertia ixx="${calf_ixx}" ixy="${calf_ixy}" ixz="${calf_ixz}" iyy="${calf_iyy}" iyz="${calf_iyz}" izz="${calf_izz}"/>
             </inertial>
         </link>
@@ -154,8 +145,5 @@
             <inertial>
                 <mass value="${foot_mass}"/>
-                <inertia
-                    ixx="${(2*foot_mass)/5.0*(foot_radius*foot_radius)}" ixy="0.0" ixz="0.0"
-                    iyy="${(2*foot_mass)/5.0*(foot_radius*foot_radius)}" iyz="0.0"
-                    izz="${(2*foot_mass)/5.0*(foot_radius*foot_radius)}"/>
+                <inertia ixx="${(2*foot_mass)/5.0*(foot_radius*foot_radius)}" ixy="0.0" ixz="0.0" iyy="${(2*foot_mass)/5.0*(foot_radius*foot_radius)}" iyz="0.0" izz="${(2*foot_mass)/5.0*(foot_radius*foot_radius)}"/>
             </inertial>
         </link>

File: robot_description/xacro/robot.xacro (robot description, xacro)
@@ -1,9 +1,10 @@
 <?xml version="1.0"?>
-<robot name="a1_description" xmlns:xacro="http://www.ros.org/wiki/xacro">
-    <xacro:include filename="$(find a1_description)/xacro/const.xacro"/>
-    <xacro:include filename="$(find a1_description)/xacro/materials.xacro"/>
-    <xacro:include filename="$(find a1_description)/xacro/leg.xacro"/>
-    <xacro:include filename="$(find a1_description)/xacro/stairs.xacro"/>
-    <xacro:include filename="$(find a1_description)/xacro/gazebo.xacro"/>
+<robot name="robot_description"
+    xmlns:xacro="http://www.ros.org/wiki/xacro">
+    <xacro:include filename="$(find robot_description)/xacro/const.xacro"/>
+    <xacro:include filename="$(find robot_description)/xacro/materials.xacro"/>
+    <xacro:include filename="$(find robot_description)/xacro/leg.xacro"/>
+    <xacro:include filename="$(find robot_description)/xacro/stairs.xacro"/>
+    <xacro:include filename="$(find robot_description)/xacro/gazebo.xacro"/>
     <xacro:if value="$(arg USE_CAMERA)">
         <xacro:include filename="$(find realsense_ros_gazebo)/xacro/depthcam.xacro"/>
@@ -11,7 +12,7 @@
     <!-- <xacro:include filename="$(find a1_gazebo)/launch/stairs.urdf.xacro"/> -->
     <!-- <xacro:stairs stairs="15" xpos="0" ypos="0" zpos="0" /> -->
-    <!-- Rollover Protection mode will add an additional stick on the top, use "true" or "false" to switch it. -->
+    <!-- rollover protection mode will add an additional stick on the top, use "true" or "false" to switch it. -->
     <xacro:property name="rolloverProtection" value="false"/>
-    <!-- Debug mode will hung up the robot, use "true" or "false" to switch it. -->
+    <!-- debug mode will hung up the robot, use "true" or "false" to switch it. -->
     <xacro:if value="$(arg DEBUG)">
         <link name="world"/>
@@ -45,5 +46,5 @@
             <origin rpy="0 0 0" xyz="0 0 0"/>
             <geometry>
-                <mesh filename="package://a1_description/meshes/trunk.dae" scale="1 1 1"/>
+                <mesh filename="package://robot_description/meshes/trunk.dae" scale="1 1 1"/>
             </geometry>
             <material name="orange"/>
@@ -58,8 +59,5 @@
             <origin rpy="0 0 0" xyz="${trunk_com_x} ${trunk_com_y} ${trunk_com_z}"/>
             <mass value="${trunk_mass}"/>
-            <inertia
-                ixx="${trunk_ixx}" ixy="${trunk_ixy}" ixz="${trunk_ixz}"
-                iyy="${trunk_iyy}" iyz="${trunk_iyz}"
-                izz="${trunk_izz}"/>
+            <inertia ixx="${trunk_ixx}" ixy="${trunk_ixy}" ixz="${trunk_ixz}" iyy="${trunk_iyy}" iyz="${trunk_iyz}" izz="${trunk_izz}"/>
         </inertial>
     </link>
@@ -91,8 +89,5 @@
             <inertial>
                 <mass value="${stick_mass}"/>
-                <inertia
-                    ixx="${stick_mass / 2.0 * (stick_radius*stick_radius)}" ixy="0.0" ixz="0.0"
-                    iyy="${stick_mass / 12.0 * (3*stick_radius*stick_radius + stick_length*stick_length)}" iyz="0.0"
-                    izz="${stick_mass / 12.0 * (3*stick_radius*stick_radius + stick_length*stick_length)}"/>
+                <inertia ixx="${stick_mass / 2.0 * (stick_radius*stick_radius)}" ixy="0.0" ixz="0.0" iyy="${stick_mass / 12.0 * (3*stick_radius*stick_radius + stick_length*stick_length)}" iyz="0.0" izz="${stick_mass / 12.0 * (3*stick_radius*stick_radius + stick_length*stick_length)}"/>
             </inertial>
         </link>

File: robot_description/xacro/transmission.xacro (robot description, xacro)
@@ -5,9 +5,9 @@
             <type>transmission_interface/SimpleTransmission</type>
             <joint name="${name}_hip_joint">
-            <hardwareInterface>hardware_interface/EffortJointInterface</hardwareInterface>
+                <hardwareInterface>hardware_interface/EffortJointInterface</hardwareInterface>
             </joint>
             <actuator name="${name}_hip_motor">
-            <hardwareInterface>hardware_interface/EffortJointInterface</hardwareInterface>
-            <mechanicalReduction>1</mechanicalReduction>
+                <hardwareInterface>hardware_interface/EffortJointInterface</hardwareInterface>
+                <mechanicalReduction>1</mechanicalReduction>
             </actuator>
         </transmission>
@@ -15,9 +15,9 @@
             <type>transmission_interface/SimpleTransmission</type>
             <joint name="${name}_thigh_joint">
-            <hardwareInterface>hardware_interface/EffortJointInterface</hardwareInterface>
+                <hardwareInterface>hardware_interface/EffortJointInterface</hardwareInterface>
             </joint>
             <actuator name="${name}_thigh_motor">
-            <hardwareInterface>hardware_interface/EffortJointInterface</hardwareInterface>
-            <mechanicalReduction>1</mechanicalReduction>
+                <hardwareInterface>hardware_interface/EffortJointInterface</hardwareInterface>
+                <mechanicalReduction>1</mechanicalReduction>
             </actuator>
         </transmission>
@@ -25,9 +25,9 @@
             <type>transmission_interface/SimpleTransmission</type>
             <joint name="${name}_calf_joint">
-            <hardwareInterface>hardware_interface/EffortJointInterface</hardwareInterface>
+                <hardwareInterface>hardware_interface/EffortJointInterface</hardwareInterface>
             </joint>
             <actuator name="${name}_calf_motor">
-            <hardwareInterface>hardware_interface/EffortJointInterface</hardwareInterface>
-            <mechanicalReduction>1</mechanicalReduction>
+                <hardwareInterface>hardware_interface/EffortJointInterface</hardwareInterface>
+                <mechanicalReduction>1</mechanicalReduction>
             </actuator>
         </transmission>
