Commit message: [hardware] add hardware commit
Signed-off-by: trantor <postrantor@gmail.com>

File: unitree_motor_example/description/ros2_control/unitree_motor.ros2_control.xacro (robot description, xacro)
@@ -2,10 +2,12 @@
 <robot xmlns:xacro="http://www.ros.org/wiki/xacro">
   <xacro:macro name="unitree_motor_control" params="name prefix use_mock_hardware">
+    <!-- @zhiqi.jia, parameters are transferred to `info_` variable in "hardware/" -->
+    <!-- include `hardware`, `joint` -->
     <ros2_control name="${name}" type="system">
       <xacro:unless value="${use_mock_hardware}">
         <hardware>
           <plugin>unitree_motor_example/UnitreeMotorSystemHardware</plugin>
-          <param name="example_param_hw_start_duration_sec">0</param>
-          <param name="example_param_hw_stop_duration_sec">3.0</param>
+          <param name="hw_start_duration_sec">0</param>
+          <param name="hw_stop_duration_sec">3.0</param>
         </hardware>
       </xacro:unless>
@@ -16,14 +18,14 @@
         </hardware>
       </xacro:if>
-      <joint name="${prefix}left_wheel_joint">
+      <joint name="${prefix}joint_ll_0_name">
         <command_interface name="velocity"/>
         <state_interface name="position"/>
         <state_interface name="velocity"/>
       </joint>
-      <joint name="${prefix}right_wheel_joint">
+      <!-- <joint name="${prefix}right_wheel_joint">
         <command_interface name="velocity"/>
         <state_interface name="position"/>
         <state_interface name="velocity"/>
-      </joint>
+      </joint> -->
     </ros2_control>
   </xacro:macro>

Commit message: [controller] modify, for unitree controller
Signed-off-by: trantor <postrantor@gmail.com>

File: unitree_motor_example/description/ros2_control/unitree_motor.ros2_control.xacro (robot description, xacro)
@@ -8,8 +8,9 @@
         <hardware>
           <plugin>unitree_motor_example/UnitreeMotorSystemHardware</plugin>
-          <param name="hw_start_duration_sec">0</param>
-          <param name="hw_stop_duration_sec">3.0</param>
+          <param name="hw_start_interval_millisec">200</param>
+          <param name="hw_stop_interval_millisec">100</param>
         </hardware>
       </xacro:unless>
+      <!-- set `false` by launch -->
       <xacro:if value="${use_mock_hardware}">
         <hardware>
@@ -18,14 +19,12 @@
         </hardware>
       </xacro:if>
+      <!-- controller_interface<->hardware_interface -->
       <joint name="${prefix}joint_ll_0_name">
         <command_interface name="velocity"/>
         <state_interface name="position"/>
         <state_interface name="velocity"/>
+        <param name="motor_id">0</param>
+        <param name="serial_port">/dev/ttyUSB0</param>
       </joint>
-      <!-- <joint name="${prefix}right_wheel_joint">
-        <command_interface name="velocity"/>
-        <state_interface name="position"/>
-        <state_interface name="velocity"/>
-      </joint> -->
     </ros2_control>
   </xacro:macro>

File: unitree_motor_example/description/urdf/unitree_motor.urdf.xacro (robot description, xacro)
@@ -8,9 +8,9 @@
   <!-- include 引入外部文件 -->
   <!-- 取决于cmake install -->
-  <xacro:include filename="$(find model_description)/unitree/urdf/unitree_motor_description.urdf.xacro" />
-  <xacro:include filename="$(find model_description)/unitree/urdf/unitree_motor.materials.xacro" />
+  <!-- <xacro:include filename="$(find model_description)/unitree/urdf/unitree_motor_description.urdf.xacro" />
+  <xacro:include filename="$(find model_description)/unitree/urdf/unitree_motor.materials.xacro" /> -->
   <xacro:include filename="$(find unitree_motor_example)/ros2_control/unitree_motor.ros2_control.xacro" />
   <!-- 实例化对象，分别在 include 中定义对应的对象 -->
-  <xacro:unitree_motor prefix="$(arg prefix)" />
+  <!-- <xacro:unitree_motor prefix="$(arg prefix)" /> -->
   <xacro:unitree_motor_control name="UnitreeMotor" prefix="$(arg prefix)" use_mock_hardware="$(arg use_mock_hardware)"/>
 </robot>

Commit message: [controller] fix hardware_interface/controller_interfaces map
Signed-off-by: Postrantor <postrantor@gmail.com>

File: unitree_motor_example/description/ros2_control/unitree_motor.ros2_control.xacro (robot description, xacro)
@@ -20,5 +20,5 @@
       </xacro:if>
       <!-- controller_interface<->hardware_interface -->
-      <joint name="${prefix}joint_ll_0_name">
+     <joint name="${prefix}joint_ll_0">
         <command_interface name="velocity"/>
         <state_interface name="position"/>

Commit message: [demo] add all
Signed-off-by: trantor <postrantor@gmail.com>

File: unitree_motor_example/description/ros2_control/unitree_motor.ros2_control.xacro (robot description, xacro)
@@ -20,5 +20,5 @@
       </xacro:if>
       <!-- controller_interface<->hardware_interface -->
-     <joint name="${prefix}joint_ll_0">
+      <joint name="${prefix}joint_ll_0">
         <command_interface name="velocity"/>
         <state_interface name="position"/>
