Commit message: [sim] try change urdf to ros2_control
Signed-off-by: trantor <postrantor@gmail.com>

File: robot_description/xacro/const.xacro (robot description, xacro)
@@ -1,4 +1,4 @@
 <?xml version="1.0"?>
-<robot name="a1_description"
+<robot name="robot_description"
     xmlns:xacro="http://www.ros.org/wiki/xacro">
     <!-- constants for robot dimensions -->
@@ -92,4 +92,5 @@
     <xacro:property name="foot_mass" value="0.06"/>
     <xacro:property name="foot_mu" value="0.8"/>
+    <!-- pid parameter -->
     <xacro:property name="kp" value="100"/>
     <xacro:property name="kd" value="1"/>

File: robot_description/xacro/gazebo.xacro (robot description, xacro)
@@ -1,49 +1,33 @@
 <?xml version="1.0"?>
 <robot>
-    <!-- ros_control plugin -->
+    <!-- <ros2_control name="GazeboSystem" type="system">
+        <hardware>
+            <plugin>gazebo_ros2_control/GazeboSystem</plugin>
+        </hardware>
+        <joint name="left_wheel_joint">
+            <command_interface name="velocity">
+                <param name="min">-1</param>
+                <param name="max">1</param>
+            </command_interface>
+            <state_interface name="position"/>
+            <state_interface name="velocity"/>
+        </joint>
+        <joint name="right_wheel_joint">
+            <command_interface name="velocity">
+                <param name="min">-1</param>
+                <param name="max">1</param>
+            </command_interface>
+            <state_interface name="position"/>
+            <state_interface name="velocity"/>
+        </joint>
+    </ros2_control> -->
+    <!-- ros2_control plugin -->
     <gazebo>
-        <plugin name="gazebo_ros_control" filename="libgazebo_ros_control.so">
-            <robotNamespace>/a1_gazebo</robotNamespace>
-            <robotSimType>gazebo_ros_control/DefaultRobotHWSim</robotSimType>
+        <plugin filename="libgazebo_ros2_control.so" name="gazebo_ros2_control">
+            <parameters>$(find robot_description)/config/controller.yaml</parameters>
+            <!-- <robotNamespace>/a1_gazebo</robotNamespace> -->
+            <!-- <robotSimType>gazebo_ros2_control/DefaultRobotHWSim</robotSimType> -->
         </plugin>
     </gazebo>
-    <!-- Show the trajectory of trunk center. -->
-    <!-- <gazebo>
-        <plugin name="3dplot" filename="libLinkPlot3DPlugin.so">
-            <frequency>10</frequency>
-            <plot>
-                <link>base</link>
-                <pose>0 0 0 0 0 0</pose>
-                <material>Gazebo/Yellow</material>
-            </plot>
-        </plugin>
-    </gazebo> -->
-    <!-- Show the trajectory of foot. You can add another trajectory about another foot. -->
-    <!-- <gazebo>
-        <plugin name="3dplot" filename="libLinkPlot3DPlugin.so">
-            <frequency>100</frequency>
-            <plot>
-                <link>FL_calf</link>
-                <pose>0 0 -0.2 0 0 0</pose>
-                <material>Gazebo/Green</material>
-            </plot>
-        </plugin>
-    </gazebo>
-    <gazebo>
-        <plugin name="3dplot" filename="libLinkPlot3DPlugin.so">
-            <frequency>100</frequency>
-            <plot>
-                <link>FR_calf</link>
-                <pose>0 0 -0.2 0 0 0</pose>
-                <material>Gazebo/Red</material>
-            </plot>
-        </plugin>
-    </gazebo> -->
-    <!-- <gazebo>
-       <plugin filename="libgazebo_ros_force.so" name="gazebo_ros_force">
-           <bodyName>trunk</bodyName>
-           <topicName>/apply_force/trunk</topicName>
-       </plugin>
-    </gazebo> -->
     <gazebo reference="imu_link">
         <gravity>true</gravity>
@@ -102,41 +86,4 @@
         </sensor>
     </gazebo>
-    <!-- visualization of foot contacts. -->
-    <!-- <gazebo reference="FR_foot">
-        <visual>
-            <plugin name="drawForcePlugin" filename="libunitreeDrawForcePlugin.so">
-                <topicName>FR_foot_contact</topicName>
-            </plugin>
-        </visual>
-    </gazebo>
-    <gazebo reference="FL_foot">
-        <visual>
-            <plugin name="drawForcePlugin" filename="libunitreeDrawForcePlugin.so">
-                <topicName>FL_foot_contact</topicName>
-            </plugin>
-        </visual>
-    </gazebo>
-    <gazebo reference="RR_foot">
-        <visual>
-            <plugin name="drawForcePlugin" filename="libunitreeDrawForcePlugin.so">
-                <topicName>RR_foot_contact</topicName>
-            </plugin>
-        </visual>
-    </gazebo>
-    <gazebo reference="RL_foot">
-        <visual>
-            <plugin name="drawForcePlugin" filename="libunitreeDrawForcePlugin.so">
-                <topicName>RL_foot_contact</topicName>
-            </plugin>
-        </visual>
-    </gazebo> -->
-    <!-- Show planned pose location -->
-    <!-- <gazebo reference="base">
-        <visual>
-            <plugin name="drawLinesPlugin" filename="libdrawLinesPlugin.so">
-                <topicName>pose_planner</topicName>
-            </plugin>
-        </visual>
-    </gazebo> -->
     <gazebo reference="base">
         <material>Gazebo/Green</material>

File: robot_description/xacro/leg.xacro (robot description, xacro)
@@ -2,6 +2,6 @@
 <robot xmlns:xacro="http://www.ros.org/wiki/xacro">
     <xacro:include filename="$(find robot_description)/xacro/transmission.xacro"/>
-    <!-- <xacro:property name="damping" value="0.3" />
-    <xacro:property name="friction" value="0.3" /> -->
+    <!-- <xacro:property name="damping" value="0.3" /> -->
+    <!-- <xacro:property name="friction" value="0.3" /> -->
     <xacro:macro name="leg" params="name mirror mirror_dae front_hind front_hind_dae *origin">
         <joint name="${name}_hip_joint" type="revolute">

File: robot_description/xacro/robot.xacro (robot description, xacro)
@@ -1,6 +1,6 @@
-<!-- ros2 run xacro xacro robot.xacro -o robot.urdf USE_CAMERA:=false DEBUG:=false -->
 <?xml version="1.0"?>
 <robot name="robot_description"
     xmlns:xacro="http://www.ros.org/wiki/xacro">
+    <!-- ros2 run xacro xacro robot.xacro -o robot.urdf USE_CAMERA:=false DEBUG:=false -->
     <xacro:include filename="$(find robot_description)/xacro/const.xacro"/>
     <xacro:include filename="$(find robot_description)/xacro/materials.xacro"/>
@@ -11,5 +11,5 @@
         <xacro:include filename="$(find realsense_ros_gazebo)/xacro/depthcam.xacro"/>
     </xacro:if>
-    <!-- <xacro:include filename="$(find a1_gazebo)/launch/stairs.urdf.xacro"/> -->
+    <!-- <xacro:include filename="$(find robot_description)/launch/stairs.urdf.xacro"/> -->
     <!-- <xacro:stairs stairs="15" xpos="0" ypos="0" zpos="0" /> -->
     <!-- rollover protection mode will add an additional stick on the top, use "true" or "false" to switch it. -->
