Commit message: [model] fix xcaro file
1. use `$(find package_name)` fix `package://`
2. remove imu.so etc.

Signed-off-by: trantor <postrantor@gmail.com>

File: robot_description/xacro/gazebo.xacro (robot description, xacro)
@@ -29,5 +29,5 @@
         </plugin>
     </gazebo>
-    <gazebo reference="imu_link">
+    <!-- <gazebo reference="imu_link">
         <gravity>true</gravity>
         <sensor name="imu_sensor" type="imu">
@@ -47,7 +47,7 @@
             <pose>0 0 0 0 0 0</pose>
         </sensor>
-    </gazebo>
+    </gazebo> -->
     <!-- Foot contacts. -->
-    <gazebo reference="FR_calf">
+    <!-- <gazebo reference="FR_calf">
         <sensor name="FR_foot_contact" type="contact">
             <update_rate>100</update_rate>
@@ -84,5 +84,5 @@
             </contact>
         </sensor>
-    </gazebo>
+    </gazebo> -->
     <gazebo reference="base">
         <material>Gazebo/Green</material>

File: robot_description/xacro/leg.xacro (robot description, xacro)
@@ -33,5 +33,5 @@
                 </xacro:if>
                 <geometry>
-                    <mesh filename="package://robot_description/meshes/hip.dae" scale="1 1 1"/>
+                    <mesh filename="$(find robot_description)/meshes/hip.dae" scale="1 1 1"/>
                 </geometry>
                 <material name="orange"/>
@@ -76,8 +76,8 @@
                 <geometry>
                     <xacro:if value="${mirror_dae == True}">
-                        <mesh filename="package://robot_description/meshes/thigh.dae" scale="1 1 1"/>
+                        <mesh filename="$(find robot_description)/meshes/thigh.dae" scale="1 1 1"/>
                     </xacro:if>
                     <xacro:if value="${mirror_dae == False}">
-                        <mesh filename="package://robot_description/meshes/thigh_mirror.dae" scale="1 1 1"/>
+                        <mesh filename="$(find robot_description)/meshes/thigh_mirror.dae" scale="1 1 1"/>
                     </xacro:if>
                 </geometry>
@@ -108,5 +108,5 @@
                 <origin rpy="0 0 0" xyz="0 0 0"/>
                 <geometry>
-                    <mesh filename="package://robot_description/meshes/calf.dae" scale="1 1 1"/>
+                    <mesh filename="$(find robot_description)/meshes/calf.dae" scale="1 1 1"/>
                 </geometry>
                 <material name="orange"/>

File: robot_description/xacro/robot.xacro (robot description, xacro)
@@ -47,5 +47,5 @@
             <origin rpy="0 0 0" xyz="0 0 0"/>
             <geometry>
-                <mesh filename="package://robot_description/meshes/trunk.dae" scale="1 1 1"/>
+                <mesh filename="$(find robot_description)/meshes/trunk.dae" scale="1 1 1"/>
             </geometry>
             <material name="orange"/>

File: robot_description/xacro/robot.xacro.urdf (robot description, URDF)
Before this commit: robot robot_a1, 23 links, 22 joints
Links:
- link FL_calf: geometry collision box size=0.13333333333333333 0.016 0.016; visual mesh filename=/home/trantor/project/model_control_ws/install/robot_descri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 scale=1 1 1
- link FL_hip: geometry collision cylinder length=0.04 radius=0.046; visual mesh filename=/home/trantor/project/model_control_ws/install/robot_descri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 scale=1 1 1
- link FL_thigh: geometry collision box size=0.2 0.0245 0.034; visual mesh filename=/home/trantor/project/model_control_ws/install/robot_descri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 scale=1 1 1
- link FR_calf: geometry collision box size=0.13333333333333333 0.016 0.016; visual mesh filename=/home/trantor/project/model_control_ws/install/robot_descri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 scale=1 1 1
- link FR_hip: geometry collision cylinder length=0.04 radius=0.046; visual mesh filename=/home/trantor/project/model_control_ws/install/robot_descri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 scale=1 1 1
- link FR_thigh: geometry collision box size=0.2 0.0245 0.034; visual mesh filename=/home/trantor/project/model_control_ws/install/robot_descri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 scale=1 1 1
- link RL_calf: geometry collision box size=0.13333333333333333 0.016 0.016; visual mesh filename=/home/trantor/project/model_control_ws/install/robot_descri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 scale=1 1 1
- link RL_hip: geometry collision cylinder length=0.04 radius=0.046; visual mesh filename=/home/trantor/project/model_control_ws/install/robot_descri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 scale=1 1 1
- link RL_thigh: geometry collision box size=0.2 0.0245 0.034; visual mesh filename=/home/trantor/project/model_control_ws/install/robot_descri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 scale=1 1 1
- link RR_calf: geometry collision box size=0.13333333333333333 0.016 0.016; visual mesh filename=/home/trantor/project/model_control_ws/install/robot_descri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 scale=1 1 1
- link RR_hip: geometry collision cylinder length=0.04 radius=0.046; visual mesh filename=/home/trantor/project/model_control_ws/install/robot_descri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 scale=1 1 1
- link RR_thigh: geometry collision box size=0.2 0.0245 0.034; visual mesh filename=/home/trantor/project/model_control_ws/install/robot_descri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 scale=1 1 1
- link trunk: geometry collision box size=0.267 0.194 0.114; visual mesh filename=/home/trantor/project/model_control_ws/install/robot_descri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 scale=1 1 1
