Commit message: [xpp] add other package, not compile
Signed-off-by: trantor <postrantor@gmail.com>

File: simulation/xpp/robots/xpp_hyq/urdf/hyq.urdf.xacro (robot description, xacro)
@@ -1,10 +1,9 @@
 <?xml version="1.0"?>
-<robot name="hyq"
-	xmlns:xacro="http://www.ros.org/wiki/xacro">
-	<xacro:property name="PI" value="3.1415926535897931"/>
-	<xacro:property name="d_lr" value="0.414"/>
-	<xacro:property name="d_fh" value="0.747"/>
-	<xacro:property name="d_tbb" value="0.082"/>
-	<xacro:property name="d_p1p2" value="0.35"/>
+<robot name="hyq" xmlns:xacro="http://www.ros.org/wiki/xacro">
+  <xacro:property name="PI" value="3.1415926535897931"/>
+  <xacro:property name="d_lr" value="0.414"/>
+  <xacro:property name="d_fh" value="0.747"/>
+  <xacro:property name="d_tbb" value="0.082"/>
+  <xacro:property name="d_p1p2" value="0.35"/>
 	<!-- HyQ trunk -->
 	<xacro:include filename="$(find xpp_hyq)/urdf/trunk.urdf.xacro"/>
@@ -15,17 +14,37 @@
 	<xacro:hyq_trunk name="base"/>
 	<!-- LF leg -->
-	<xacro:hyq_leg name="lf" parent="trunk" reflect_hip="1" reflect_upper="1" reflect_front="1">
+	<xacro:hyq_leg
+		name="lf"
+		parent="trunk"
+		reflect_hip="1"
+		reflect_upper="1"
+		reflect_front="1">
 		<origin xyz="${d_fh/2} ${d_lr/2} 0" rpy="0 ${PI/2} ${PI}"/>
 	</xacro:hyq_leg>
 	<!-- RF leg -->
-	<xacro:hyq_leg name="rf" parent="trunk" reflect_hip="-1" reflect_upper="-1" reflect_front="1">
+	<xacro:hyq_leg
+		name="rf"
+		parent="trunk"
+		reflect_hip="-1"
+		reflect_upper="-1"
+		reflect_front="1">
 		<origin xyz="${d_fh/2} ${-d_lr/2} 0" rpy="0 ${PI/2} 0"/>
 	</xacro:hyq_leg>
 	<!-- LH leg -->
-	<xacro:hyq_leg name="lh" parent="trunk" reflect_hip="-1" reflect_upper="1" reflect_front="-1">
+	<xacro:hyq_leg
+		name="lh"
+		parent="trunk"
+		reflect_hip="-1"
+		reflect_upper="1"
+		reflect_front="-1">
 		<origin xyz="${-d_fh/2} ${d_lr/2} 0" rpy="0 ${PI/2} ${PI}"/>
 	</xacro:hyq_leg>
 	<!-- RH leg -->
-	<xacro:hyq_leg name="rh" parent="trunk" reflect_hip="1" reflect_upper="-1" reflect_front="-1">
+	<xacro:hyq_leg
+		name="rh"
+		parent="trunk"
+		reflect_hip="1"
+		reflect_upper="-1"
+		reflect_front="-1">
 		<origin xyz="${-d_fh/2} ${-d_lr/2} 0" rpy="0 ${PI/2} 0"/>
 	</xacro:hyq_leg>

File: simulation/xpp/robots/xpp_hyq/urdf/leg.urdf.xacro (robot description, xacro)
@@ -8,5 +8,5 @@
 			<xacro:insert_block name="origin"/>
 			<parent link="${parent}"/>
-			<child link="${name}_hipassembly"/>
+			<child  link="${name}_hipassembly"/>
 			<axis xyz="0 0 1"/>
 			<limit effort="150.0" velocity="12.0" lower="${-7*PI/18}" upper="${PI/6}"/>
@@ -16,7 +16,9 @@
 			<origin xyz="${d_tbb} 0 0" rpy="${reflect_upper*PI/2} 0 0"/>
 			<parent link="${name}_hipassembly"/>
-			<child link="${name}_upperleg"/>
+			<child  link="${name}_upperleg"/>
 			<axis xyz="0 0 1"/>
-			<limit effort="150.0" velocity="12.0" lower="${-(1+reflect_front)*5*PI/36-(1-reflect_front)*7*PI/36}" upper="${(1-reflect_front)*5*PI/36+(1+reflect_front)*7*PI/36}"/>
+			<limit effort="150.0" velocity="12.0"
+          lower="${-(1+reflect_front)*5*PI/36-(1-reflect_front)*7*PI/36}"
+          upper="${(1-reflect_front)*5*PI/36+(1+reflect_front)*7*PI/36}"/>
 		</joint>
 		<!-- Lower leg joint -->
@@ -24,7 +26,9 @@
 			<origin xyz="${d_p1p2} 0 0" rpy="0 0 0"/>
 			<parent link="${name}_upperleg"/>
-			<child link="${name}_lowerleg"/>
+			<child  link="${name}_lowerleg"/>
 			<axis xyz="0 0 1"/>
-			<limit effort="150.0" velocity="12.0" lower="${-(1+reflect_front)*7*PI/18+(1-reflect_front)*PI/18}" upper="${(1-reflect_front)*7*PI/18-(1+reflect_front)*PI/18}"/>
+			<limit effort="150.0" velocity="12.0"
+          lower="${-(1+reflect_front)*7*PI/18+(1-reflect_front)*PI/18}"
+          upper="${(1-reflect_front)*7*PI/18-(1+reflect_front)*PI/18}"/>
 		</joint>
 		<!-- Foot joint -->
@@ -32,5 +36,5 @@
 			<origin xyz="0.35 0 0" rpy="${PI/2} 0 ${-PI/2}"/>
 			<parent link="${name}_lowerleg"/>
-			<child link="${name}_foot"/>
+			<child  link="${name}_foot"/>
 		</joint>
 		<!-- Links -->
