Commit message: [simulation] fix robot.xacro file
- remote `use_camera`
- add `use_mock_hardware`
- remove stairs.xacro
- delete spawn.launch
- set xacro gazebo tag

Signed-off-by: trantor <postrantor@gmail.com>

File: simulation/robot_description/config/ros2_control.xacro (robot description, xacro)
@@ -1,136 +1,145 @@
 <?xml version="1.0"?>
-<robot name="robot_a1"
-  xmlns:xacro="http://www.ros.org/wiki/xacro">
-  <ros2_control name="GazeboSystem" type="system">
-    <hardware>
-      <plugin>gazebo_ros2_control/GazeboSystem</plugin>
-    </hardware>
-    <xacro:unless value="${use_mock_hardware}">
-      <hardware>
-        <plugin>unitree_motor_example/UnitreeMotorSystemHardware</plugin>
-        <param name="hw_start_interval_millisec">200</param>
-        <param name="hw_stop_interval_millisec">100</param>
-      </hardware>
-    </xacro:unless>
-    <joint name="FL_hip_joint">
-      <command_interface name="velocity">
-        <param name="min">-1</param>
-        <param name="max">1</param>
-      </command_interface>
-      <state_interface name="position"/>
-      <state_interface name="velocity"/>
-      <param name="motor_id">0</param>
-      <param name="serial_port">/dev/ttyUSB0</param>
-    </joint>
-    <joint name="FL_thigh_joint">
-      <command_interface name="velocity">
-        <param name="min">-1</param>
-        <param name="max">1</param>
-      </command_interface>
-      <state_interface name="position"/>
-      <state_interface name="velocity"/>
-      <param name="motor_id">1</param>
-      <param name="serial_port">/dev/ttyUSB0</param>
-    </joint>
-    <joint name="FL_calf_joint">
-      <command_interface name="velocity">
-        <param name="min">-1</param>
-        <param name="max">1</param>
-      </command_interface>
-      <state_interface name="position"/>
-      <state_interface name="velocity"/>
-      <param name="motor_id">2</param>
-      <param name="serial_port">/dev/ttyUSB0</param>
-    </joint>
-    <joint name="FR_hip_joint">
-      <command_interface name="velocity">
-        <param name="min">-1</param>
-        <param name="max">1</param>
-      </command_interface>
-      <state_interface name="position"/>
-      <state_interface name="velocity"/>
-      <param name="motor_id">3</param>
-      <param name="serial_port">/dev/ttyUSB0</param>
-    </joint>
-    <joint name="FR_thigh_joint">
-      <command_interface name="velocity">
-        <param name="min">-1</param>
-        <param name="max">1</param>
-      </command_interface>
-      <state_interface name="position"/>
-      <state_interface name="velocity"/>
-      <param name="motor_id">4</param>
-      <param name="serial_port">/dev/ttyUSB0</param>
-    </joint>
-    <joint name="FR_calf_joint">
-      <command_interface name="velocity">
-        <param name="min">-1</param>
-        <param name="max">1</param>
-      </command_interface>
-      <state_interface name="position"/>
-      <state_interface name="velocity"/>
-      <param name="motor_id">5</param>
-      <param name="serial_port">/dev/ttyUSB0</param>
-    </joint>
-    <joint name="RL_hip_joint">
-      <command_interface name="velocity">
-        <param name="min">-1</param>
-        <param name="max">1</param>
-      </command_interface>
-      <state_interface name="position"/>
-      <state_interface name="velocity"/>
-      <param name="motor_id">6</param>
-      <param name="serial_port">/dev/ttyUSB0</param>
-    </joint>
-    <joint name="RL_thigh_joint">
-      <command_interface name="velocity">
-        <param name="min">-1</param>
-        <param name="max">1</param>
-      </command_interface>
-      <state_interface name="position"/>
-      <state_interface name="velocity"/>
-      <param name="motor_id">7</param>
-      <param name="serial_port">/dev/ttyUSB0</param>
-    </joint>
-    <joint name="RL_calf_joint">
-      <command_interface name="velocity">
-        <param name="min">-1</param>
-        <param name="max">1</param>
-      </command_interface>
-      <state_interface name="position"/>
-      <state_interface name="velocity"/>
-      <param name="motor_id">8</param>
-      <param name="serial_port">/dev/ttyUSB0</param>
-    </joint>
-    <joint name="RR_hip_joint">
-      <command_interface name="velocity">
-        <param name="min">-1</param>
-        <param name="max">1</param>
-      </command_interface>
-      <state_interface name="position"/>
-      <state_interface name="velocity"/>
-      <param name="motor_id">9</param>
-      <param name="serial_port">/dev/ttyUSB0</param>
-    </joint>
-    <joint name="RR_thigh_joint">
-      <command_interface name="velocity">
-        <param name="min">-1</param>
-        <param name="max">1</param>
-      </command_interface>
-      <state_interface name="position"/>
-      <state_interface name="velocity"/>
-      <param name="motor_id">10</param>
-      <param name="serial_port">/dev/ttyUSB0</param>
-    </joint>
-    <joint name="RR_calf_joint">
-      <command_interface name="velocity">
-        <param name="min">-1</param>
-        <param name="max">1</param>
-      </command_interface>
-      <state_interface name="position"/>
-      <state_interface name="velocity"/>
-      <param name="motor_id">11</param>
-      <param name="serial_port">/dev/ttyUSB0</param>
-    </joint>
-  </ros2_control>
+<robot xmlns:xacro="http://www.ros.org/wiki/xacro">
+  <xacro:macro name="use_ros2_control" params="use_mock_hardware">
+    <ros2_control name="GazeboSystem" type="system">
+      <!-- set `false` by launch -->
+      <xacro:if value="${use_mock_hardware}">
+        <hardware>
+          <plugin>gazebo_ros2_control/GazeboSystem</plugin>
+        </hardware>
+      </xacro:if>
+      <xacro:unless value="${use_mock_hardware}">
+        <hardware>
+          <plugin>unitree_motor_example/UnitreeMotorSystemHardware</plugin>
+          <param name="hw_start_interval_millisec">200</param>
+          <param name="hw_stop_interval_millisec">100</param>
+        </hardware>
+      </xacro:unless>
+      <!-- controller_interface<->hardware_interface -->
+      <!-- FL_joint -->
+      <joint name="FL_hip_joint">
+        <command_interface name="velocity">
+          <param name="min">-1</param>
+          <param name="max">1</param>
+        </command_interface>
+        <state_interface name="position"/>
+        <state_interface name="velocity"/>
+        <param name="motor_id">0</param>
+        <param name="serial_port">/dev/ttyUSB0</param>
+      </joint>
+      <joint name="FL_thigh_joint">
+        <command_interface name="velocity">
+          <param name="min">-1</param>
+          <param name="max">1</param>
+        </command_interface>
+        <state_interface name="position"/>
+        <state_interface name="velocity"/>
+        <param name="motor_id">1</param>
+        <param name="serial_port">/dev/ttyUSB0</param>
+      </joint>
+      <joint name="FL_calf_joint">
+        <command_interface name="velocity">
+          <param name="min">-1</param>
+          <param name="max">1</param>
+        </command_interface>
+        <state_interface name="position"/>
+        <state_interface name="velocity"/>
+        <param name="motor_id">2</param>
+        <param name="serial_port">/dev/ttyUSB0</param>
+      </joint>
+      <!-- FR_joint -->
+      <joint name="FR_hip_joint">
+        <command_interface name="velocity">
+          <param name="min">-1</param>
+          <param name="max">1</param>
+        </command_interface>
+        <state_interface name="position"/>
+        <state_interface name="velocity"/>
+        <param name="motor_id">3</param>
+        <param name="serial_port">/dev/ttyUSB0</param>
+      </joint>
+      <joint name="FR_thigh_joint">
+        <command_interface name="velocity">
+          <param name="min">-1</param>
+          <param name="max">1</param>
+        </command_interface>
+        <state_interface name="position"/>
+        <state_interface name="velocity"/>
+        <param name="motor_id">4</param>
+        <param name="serial_port">/dev/ttyUSB0</param>
+      </joint>
+      <joint name="FR_calf_joint">
+        <command_interface name="velocity">
+          <param name="min">-1</param>
+          <param name="max">1</param>
+        </command_interface>
+        <state_interface name="position"/>
+        <state_interface name="velocity"/>
+        <param name="motor_id">5</param>
+        <param name="serial_port">/dev/ttyUSB0</param>
+      </joint>
+      <!-- RL_joint -->
+      <joint name="RL_hip_joint">
+        <command_interface name="velocity">
+          <param name="min">-1</param>
+          <param name="max">1</param>
+        </command_interface>
+        <state_interface name="position"/>
+        <state_interface name="velocity"/>
+        <param name="motor_id">6</param>
+        <param name="serial_port">/dev/ttyUSB0</param>
+      </joint>
+      <joint name="RL_thigh_joint">
+        <command_interface name="velocity">
+          <param name="min">-1</param>
+          <param name="max">1</param>
+        </command_interface>
+        <state_interface name="position"/>
+        <state_interface name="velocity"/>
+        <param name="motor_id">7</param>
+        <param name="serial_port">/dev/ttyUSB0</param>
+      </joint>
+      <joint name="RL_calf_joint">
+        <command_interface name="velocity">
+          <param name="min">-1</param>
+          <param name="max">1</param>
+        </command_interface>
+        <state_interface name="position"/>
+        <state_interface name="velocity"/>
+        <param name="motor_id">8</param>
+        <param name="serial_port">/dev/ttyUSB0</param>
+      </joint>
+      <!-- RR_joint -->
+      <joint name="RR_hip_joint">
+        <command_interface name="velocity">
+          <param name="min">-1</param>
+          <param name="max">1</param>
+        </command_interface>
+        <state_interface name="position"/>
+        <state_interface name="velocity"/>
+        <param name="motor_id">9</param>
+        <param name="serial_port">/dev/ttyUSB0</param>
+      </joint>
+      <joint name="RR_thigh_joint">
+        <command_interface name="velocity">
+          <param name="min">-1</param>
+          <param name="max">1</param>
+        </command_interface>
+        <state_interface name="position"/>
+        <state_interface name="velocity"/>
+        <param name="motor_id">10</param>
+        <param name="serial_port">/dev/ttyUSB0</param>
+      </joint>
+      <joint name="RR_calf_joint">
+        <command_interface name="velocity">
+          <param name="min">-1</param>
+          <param name="max">1</param>
+        </command_interface>
+        <state_interface name="position"/>
+        <state_interface name="velocity"/>
+        <param name="motor_id">11</param>
+        <param name="serial_port">/dev/ttyUSB0</param>
+      </joint>
+    </ros2_control>
+  </xacro:macro>
 </robot>

File: simulation/robot_description/xacro/gazebo.xacro (robot description, xacro)
@@ -1,9 +1,15 @@
 <?xml version="1.0"?>
-<robot>
+<robot name="robot_a1"
+    xmlns:xacro="http://www.ros.org/wiki/xacro">
     <gazebo>
         <plugin filename="libgazebo_ros2_control.so" name="gazebo_ros2_control">
             <parameters>$(find robot_description)/config/controller.yaml</parameters>
-            <robotNamespace>/a1_gazebo</robotNamespace>
-            <robotSimType>gazebo_ros2_control/DefaultRobotHWSim</robotSimType>
+            <robot_param>robot_description</robot_param>
+            <robot_param_node>robot_state_publisher</robot_param_node>
+            <ros>
+                <!-- <namespace>/robot_a1</namespace> -->
+                <!-- <remapping>/old_topic:=/new_topic</remapping> -->
+                <!-- <remapping>/another_old_topic:=/another_new_topic</remapping> -->
+            </ros>
         </plugin>
     </gazebo>

File: simulation/robot_description/xacro/leg.xacro (robot description, xacro)
@@ -1,4 +1,5 @@
 <?xml version="1.0"?>
-<robot xmlns:xacro="http://www.ros.org/wiki/xacro">
+<robot name="robot_a1"
+    xmlns:xacro="http://www.ros.org/wiki/xacro">
     <xacro:include filename="$(find robot_description)/xacro/transmission.xacro"/>
     <!-- <xacro:property name="damping" value="0.3" /> -->

File: simulation/robot_description/xacro/robot.xacro (robot description, xacro)
@@ -2,20 +2,16 @@
 <robot name="robot_a1"
     xmlns:xacro="http://www.ros.org/wiki/xacro">
-    <!-- ros2 run xacro xacro robot.xacro -o robot.urdf USE_CAMERA:=false DEBUG:=false -->
     <xacro:include filename="$(find robot_description)/xacro/const.xacro"/>
     <xacro:include filename="$(find robot_description)/xacro/materials.xacro"/>
     <xacro:include filename="$(find robot_description)/xacro/leg.xacro"/>
-    <xacro:include filename="$(find robot_description)/xacro/stairs.xacro"/>
     <xacro:include filename="$(find robot_description)/xacro/gazebo.xacro"/>
+    <!-- <xacro:include filename="$(find robot_description)/xacro/stairs.xacro"/> -->
+    <!-- <xacro:stairs stairs="15" xpos="0" ypos="0" zpos="0" /> -->
     <xacro:include filename="$(find robot_description)/config/ros2_control.xacro"/>
-    <xacro:if value="$(arg USE_CAMERA)">
-        <xacro:include filename="$(find realsense_ros_gazebo)/xacro/depthcam.xacro"/>
-    </xacro:if>
-    <!-- <xacro:include filename="$(find robot_description)/launch/stairs.urdf.xacro"/> -->
-    <!-- <xacro:stairs stairs="15" xpos="0" ypos="0" zpos="0" /> -->
+    <xacro:use_ros2_control use_mock_hardware="$(arg use_mock_hardware)" />
     <!-- rollover protection mode will add an additional stick on the top, use "true" or "false" to switch it. -->
     <xacro:property name="rolloverProtection" value="false"/>
     <!-- debug mode will hung up the robot, use "true" or "false" to switch it. -->
-    <xacro:if value="$(arg DEBUG)">
+    <xacro:if value="$(arg debug)">
         <link name="world"/>
         <joint name="base_static_joint" type="fixed">
@@ -64,9 +60,4 @@
         </inertial>
     </link>
-    <xacro:if value="$(arg USE_CAMERA)">
-        <xacro:realsense_d435 sensor_name="d435" parent_link="trunk" rate="10">
-            <origin rpy="0 0 0 " xyz="0.25 0 0.055"/>
-        </xacro:realsense_d435>
-    </xacro:if>
     <xacro:if value="${(rolloverProtection == 'true')}">
         <joint name="stick_joint" type="fixed">
