Commit message: [launch] refactor robot_description
Signed-off-by: trantor <postrantor@gmail.com>

File: simulation/robot_description/config/controller/ros2_control.xacro (robot description, xacro)
@@ -1,4 +1,16 @@
 <?xml version="1.0"?>
 <robot xmlns:xacro="http://www.ros.org/wiki/xacro">
+  <gazebo>
+    <plugin filename="libgazebo_ros2_control.so" name="gazebo_ros2_control">
+      <parameters>$(find robot_description)/config/controller/controller.yaml</parameters>
+      <robot_param>robot_description</robot_param>
+      <robot_param_node>robot_state_publisher</robot_param_node>
+      <ros>
+        <!-- <namespace>/robot_a1</namespace> -->
+        <!-- <remapping>/old_topic:=/new_topic</remapping> -->
+        <!-- <remapping>/another_old_topic:=/another_new_topic</remapping> -->
+      </ros>
+    </plugin>
+  </gazebo>
   <xacro:macro name="use_ros2_control" params="use_mock_hardware">
     <ros2_control name="GazeboSystem" type="system">

File: simulation/robot_description/config/xacro/gazebo.xacro (robot description, xacro)
@@ -2,16 +2,4 @@
 <robot name="robot_a1"
     xmlns:xacro="http://www.ros.org/wiki/xacro">
-    <gazebo>
-        <plugin filename="libgazebo_ros2_control.so" name="gazebo_ros2_control">
-            <parameters>$(find robot_description)/config/controller.yaml</parameters>
-            <robot_param>robot_description</robot_param>
-            <robot_param_node>robot_state_publisher</robot_param_node>
-            <ros>
-                <!-- <namespace>/robot_a1</namespace> -->
-                <!-- <remapping>/old_topic:=/new_topic</remapping> -->
-                <!-- <remapping>/another_old_topic:=/another_new_topic</remapping> -->
-            </ros>
-        </plugin>
-    </gazebo>
     <!-- <gazebo reference="imu_link">
         <gravity>true</gravity>

File: simulation/robot_description/config/xacro/leg.xacro (robot description, xacro)
@@ -2,5 +2,5 @@
 <robot name="robot_a1"
     xmlns:xacro="http://www.ros.org/wiki/xacro">
-    <xacro:include filename="$(find robot_description)/xacro/transmission.xacro"/>
+    <xacro:include filename="$(find robot_description)/config/xacro/transmission.xacro"/>
     <!-- <xacro:property name="damping" value="0.3" /> -->
     <!-- <xacro:property name="friction" value="0.3" /> -->
@@ -34,5 +34,5 @@
                 </xacro:if>
                 <geometry>
-                    <mesh filename="$(find robot_description)/meshes/hip.dae" scale="1 1 1"/>
+                    <mesh filename="$(find robot_description)/config/meshes/hip.dae" scale="1 1 1"/>
                 </geometry>
                 <material name="orange"/>
@@ -77,8 +77,8 @@
                 <geometry>
                     <xacro:if value="${mirror_dae == True}">
-                        <mesh filename="$(find robot_description)/meshes/thigh.dae" scale="1 1 1"/>
+                        <mesh filename="$(find robot_description)/config/meshes/thigh.dae" scale="1 1 1"/>
                     </xacro:if>
                     <xacro:if value="${mirror_dae == False}">
-                        <mesh filename="$(find robot_description)/meshes/thigh_mirror.dae" scale="1 1 1"/>
+                        <mesh filename="$(find robot_description)/config/meshes/thigh_mirror.dae" scale="1 1 1"/>
                     </xacro:if>
                 </geometry>
@@ -109,5 +109,5 @@
                 <origin rpy="0 0 0" xyz="0 0 0"/>
                 <geometry>
-                    <mesh filename="$(find robot_description)/meshes/calf.dae" scale="1 1 1"/>
+                    <mesh filename="$(find robot_description)/config/meshes/calf.dae" scale="1 1 1"/>
                 </geometry>
                 <material name="orange"/>

File: simulation/robot_description/config/xacro/robot.xacro (robot description, xacro)
@@ -2,11 +2,11 @@
 <robot name="robot_a1"
     xmlns:xacro="http://www.ros.org/wiki/xacro">
-    <xacro:include filename="$(find robot_description)/xacro/const.xacro"/>
-    <xacro:include filename="$(find robot_description)/xacro/materials.xacro"/>
-    <xacro:include filename="$(find robot_description)/xacro/leg.xacro"/>
-    <xacro:include filename="$(find robot_description)/xacro/gazebo.xacro"/>
-    <!-- <xacro:include filename="$(find robot_description)/xacro/stairs.xacro"/> -->
+    <xacro:include filename="$(find robot_description)/config/controller/ros2_control.xacro"/>
+    <xacro:include filename="$(find robot_description)/config/xacro/const.xacro"/>
+    <xacro:include filename="$(find robot_description)/config/xacro/materials.xacro"/>
+    <xacro:include filename="$(find robot_description)/config/xacro/leg.xacro"/>
+    <xacro:include filename="$(find robot_description)/config/xacro/gazebo.xacro"/>
+    <!-- <xacro:include filename="$(find robot_description)/config/xacro/stairs.xacro"/> -->
     <!-- <xacro:stairs stairs="15" xpos="0" ypos="0" zpos="0" /> -->
-    <xacro:include filename="$(find robot_description)/config/ros2_control.xacro"/>
     <xacro:use_ros2_control use_mock_hardware="$(arg use_mock_hardware)" />
     <!-- rollover protection mode will add an additional stick on the top, use "true" or "false" to switch it. -->
@@ -44,5 +44,5 @@
             <origin rpy="0 0 0" xyz="0 0 0"/>
             <geometry>
-                <mesh filename="$(find robot_description)/meshes/trunk.dae" scale="1 1 1"/>
+                <mesh filename="$(find robot_description)/config/meshes/trunk.dae" scale="1 1 1"/>
             </geometry>
             <material name="orange"/>
